Commit message: Added right front caster link and joint

File: urdf/teztecbot_rearpowered.urdf (robot description, URDF)
Before this commit: robot teztecbot, 1 links, 0 joints
Links:
- added link front_right_caster_link, mass 0.0; collision box size=0.075 0.01 0.075; visual box size=0.075 0.01 0.075
- link base_link: mass 0.0 -> 5.0; geometry collision box size=0.575 0.575 0.35; visual box size=0.575 0.575 0.35
Joints:
- added joint front_right_caster_joint: type continuous, parent base_link, child front_right_caster_link, origin xyz=0.1375 0.2875 -0.175 rpy=0.0 0.0 0.0, axis 0.0 0.0 1, limit lower=0.0 upper=0.0 effort=0.0 velocity=0.0

Commit message: Added left front caster link and joint

File: urdf/teztecbot_rearpowered.urdf (robot description, URDF)
Before this commit: robot teztecbot, 2 links, 1 joints
Links:
- added link front_left_caster_link, mass 0.0; collision box size=0.075 0.01 0.075; visual box size=0.075 0.01 0.075
Joints:
- added joint front_left_caster_joint: type continuous, parent base_link, child front_left_caster_link, origin xyz=0.1375 0.2875 -0.175 rpy=0.0 0.0 0.0, axis 0.0 0.0 1, limit lower=0.0 upper=0.0 effort=0.0 velocity=0.0
- joint front_right_caster_joint: origin xyz=0.1375 0.2875 -0.175 rpy=0.0 0.0 0.0 -> xyz=0.1375 -0.2875 -0.175 rpy=0.0 0.0 0.0

Commit message: Fixed front caster link and joint

File: urdf/teztecbot_rearpowered.urdf (robot description, URDF)
Before this commit: robot teztecbot, 3 links, 2 joints
Links:
- removed link front_left_caster_link
- added link front_right_wheel_link, mass 0.0; collision cylinder length=0.05 radius=0.15; visual cylinder length=0.05 radius=0.075
Joints:
- removed joint front_left_caster_joint
- added joint front_right_wheel_joint: type continuous, parent front_right_caster_link, child front_right_wheel_link, origin xyz=0.075 0.0 -0.075 rpy=-1.5708 0.0 0.0, axis 0.0 0.0 1, limit lower=0.0 upper=0.0 effort=0.0 velocity=0.0

Commit message: Added right front caster link and joint

File: urdf/teztecbot_rearpowered.urdf (robot description, URDF)
Before this commit: robot teztecbot, 3 links, 2 joints
Links:
- added link front_left_caster_link, mass 0.0; collision box size=0.075 0.01 0.075; visual box size=0.075 0.01 0.075
- added link front_left_wheel_link, mass 0.0; collision cylinder length=0.05 radius=0.15; visual cylinder length=0.05 radius=0.075
Joints:
- added joint front_left_caster_joint: type continuous, parent base_link, child front_left_caster_link, origin xyz=0.1375 0.2875 -0.175 rpy=0.0 0.0 0.0, axis 0.0 0.0 1, limit lower=0.0 upper=0.0 effort=0.0 velocity=0.0
- added joint front_left_wheel_joint: type continuous, parent front_left_caster_link, child front_left_wheel_link, origin xyz=0.075 0.0 -0.075 rpy=-1.5708 0.0 0.0, axis 0.0 0.0 1, limit lower=0.0 upper=0.0 effort=0.0 velocity=0.0

Commit message: Added right rear wheel

File: urdf/teztecbot_rearpowered.urdf (robot description, URDF)
Before this commit: robot teztecbot, 5 links, 4 joints
Links:
- added link right_wheel_link, mass 0.0; collision cylinder length=0.02 radius=0.10; visual cylinder length=0.02 radius=0.10
- link front_left_wheel_link: geometry collision cylinder length=0.05 radius=0.075; visual cylinder length=0.05 radius=0.075
- link front_right_wheel_link: geometry collision cylinder length=0.05 radius=0.075; visual cylinder length=0.05 radius=0.075
Joints:
- added joint right_wheel_joint: type continuous, parent base_link, child right_wheel_link, origin xyz=-0.1875 -0.2875 -0.225 rpy=-1.5708 0.0 0.0, axis 0.0 0.0 1, limit lower=0.0 upper=0.0 effort=0.0 velocity=0.0

Commit message: Added left rear wheel

File: urdf/teztecbot_rearpowered.urdf (robot description, URDF)
Before this commit: robot teztecbot, 6 links, 5 joints
Links:
- added link left_wheel_link, mass 0.0; collision cylinder length=0.02 radius=0.10; visual cylinder length=0.02 radius=0.10
Joints:
- added joint left_wheel_joint: type continuous, parent base_link, child left_wheel_link, origin xyz=-0.1875 0.2875 -0.225 rpy=-1.5708 0.0 0.0, axis 0.0 0.0 1, limit lower=0.0 upper=0.0 effort=0.0 velocity=0.0

Commit message: Added rgbd representation

File: urdf/teztecbot_rearpowered.urdf (robot description, URDF)
Before this commit: robot teztecbot, 7 links, 6 joints
Links:
- added link rgbd_cam_link, mass 0.0; collision box size=0.025 0.25 0.05; visual box size=0.025 0.25 0.05
Joints:
- added joint rgbd_cam_joint: type fixed, parent base_link, child rgbd_cam_link, origin xyz=0.275 0.0 0.2 rpy=0.0 0.0 0.0, axis 0.0 0.0 0.0, limit lower=0.0 upper=0.0 effort=0.0 velocity=0.0

Commit message: Added mass to all links

File: urdf/teztecbot_rearpowered.urdf (robot description, URDF)
Before this commit: robot teztecbot, 8 links, 7 joints
Links:
- link front_left_caster_link: mass 0.0 -> 0.5
- link front_left_wheel_link: mass 0.0 -> 1.0
- link front_right_caster_link: mass 0.0 -> 0.5
- link front_right_wheel_link: mass 0.0 -> 1.0
- link left_wheel_link: mass 0.0 -> 1.5
- link rgbd_cam_link: mass 0.0 -> 0.1
- link right_wheel_link: mass 0.0 -> 1.5

Commit message: Fixed wheels dimentions

File: urdf/teztecbot_rearpowered.urdf (robot description, URDF)
Before this commit: robot teztecbot, 8 links, 7 joints
Links:
- link front_left_wheel_link: geometry collision cylinder length=0.02 radius=0.075; visual cylinder length=0.02 radius=0.075
- link front_right_wheel_link: geometry collision cylinder length=0.02 radius=0.075; visual cylinder length=0.02 radius=0.075
- link left_wheel_link: geometry collision cylinder length=0.05 radius=0.10; visual cylinder length=0.05 radius=0.10
- link right_wheel_link: geometry collision cylinder length=0.05 radius=0.10; visual cylinder length=0.05 radius=0.10

Commit message: Fixed inertias again

File: urdf/teztecbot_rearpowered.urdf (robot description, URDF)
Before this commit: robot teztecbot, 8 links, 7 joints
Links:
- link front_left_caster_link: mass 0.5 -> 0.2
- link front_left_wheel_link: mass 1.0 -> 1
- link front_right_caster_link: mass 0.5 -> 0.2
- link front_right_wheel_link: mass 1.0 -> 1

Commit message: Rotated coasters for a better performance al beginin in the rearpowered version

File: urdf/teztecbot_rearpowered.urdf (robot description, URDF)
Before this commit: robot teztecbot, 8 links, 7 joints
Joints:
- joint front_left_caster_joint: origin xyz=0.1375 0.2875 -0.175 rpy=0.0 0.0 0.0 -> xyz=0.1375 0.2875 -0.175 rpy=0.0 0.0 3.14159
- joint front_right_caster_joint: origin xyz=0.1375 -0.2875 -0.175 rpy=0.0 0.0 0.0 -> xyz=0.1375 -0.2875 -0.175 rpy=0.0 0.0 3.14159
