Commit message: Rotated casters for a better performance at beginin

File: urdf/teztecbot_frontpowered.urdf (robot description, URDF)
Before this commit: robot teztecbot, 8 links, 7 joints
Joints:
- joint back_left_caster_joint: origin xyz=-0.1375 0.2875 -0.175 rpy=0.0 0.0 0.0 -> xyz=-0.1375 0.2875 -0.175 rpy=0.0 0.0 3.14159
- joint back_right_caster_joint: origin xyz=-0.1375 -0.2875 -0.175 rpy=0.0 0.0 0.0 -> xyz=-0.1375 -0.2875 -0.175 rpy=0.0 0.0 3.14159

Commit message: Fixed library that doesnt use gpu for laser sensor

File: urdf/teztecbot_frontpowered.urdf (robot description, URDF)
Before this commit: robot teztecbot, 8 links, 7 joints
Links:
- link base_link: mass 5.0 -> None
