Commit message: Decremented the height of the ramps

File: urdf/platform.urdf.xacro (robot description, xacro)
@@ -4,5 +4,5 @@
     <xacro:property name="B"        value="5.0" />
     <xacro:property name="C"        value="1.0" />
-    <xacro:property name="C_O"      value="0.3" />
+    <xacro:property name="C_O"      value="0.2" />
     <xacro:property name="alpha"    value="${20*pi/180}" />
     <xacro:property name="x_adj"    value="0.6" />
